File: current_protection.kicad_sch (KiCad schematic)
At the start: 0 parts

Commit message: Finished 5V buck converter schematic
Other:
- company: (none) -> Longhorn Racing Solar
Changed lines of the file:
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@@
 	(generator_version "8.0")
 	(paper "A4")
+	(title_block
+		(company "Longhorn Racing Solar")
+		(comment 1 "https://cloud.wikis.utexas.edu/wiki/x/-qKvAQ")
+	)
+	(hierarchical_label "5V_IN"
+		(shape input)
+		(at 102.87 88.9 0)
+		(fields_autoplaced yes)
+		(effects
+			(font
+				(size 1.27 1.27)
+			)
+			(justify left)
+		)
+	)
+	(hierarchical_label "12V_IN"
+		(shape input)
+		(at 102.87 83.82 0)
+		(fields_autoplaced yes)
+		(effects
+			(font
+				(size 1.27 1.27)
+			)
+			(justify left)
+		)
+	)
 )
