File: USBCPowerPCB.kicad_pcb (KiCad board)
At the start: 4 copper layers, 112 parts, among them IC1 TPS56A37RPAR, IC2 NPS4053GVH, J1 USB_C_Receptacle_PowerOnly_6P, J10 GND_BANANA_OUT, J2 CC, J3 12V_OUT, J4 5V_ISOOUT, J5 5V_UNISOOUT, J6 12V_OUT_PIN, J7 5V_ISOOUT_PIN, J8 5V_UNISOOUT_PIN, J9 12V_BANANA_OUT, Q1 IRF9358TRPBF, Q2 BSL308PEH6327XTSA1, Q3 NVTR4503NT1G, Q4 SI7149ADP-T1-GE3, Q5 SI7149ADP-T1-GE3, U1 TVS2200DRV, U2 CYPD3177-24LQXQT, U3 MAX16914AUB+, U4 TPS562231DRLR, U5 TPS2116DRL, U6 TBA2-2411

Commit message: Addressed most of the review comments, fixed power protection, added bigger caps & better part selection on 12V and 5V out, changed 5V buck inductor, fixed power good & fault LEDs
Parts:
- removed C1, C2: 3.3uF, Capacitor_SMD:C_0805_2012Metric
- removed C10, C18, C9: 10uF, Capacitor_SMD:C_2220_5750Metric
- removed C11, C13, C15, C19, C21, C4, C5: 0.1uF, Capacitor_SMD:C_0805_2012Metric
- removed C12: DNP, Capacitor_SMD:C_0805_2012Metric
- removed C14: 33pF, Capacitor_SMD:C_0805_2012Metric
- removed C16, C17, C20, C22: 22uF, Capacitor_SMD:C_0805_2012Metric
- removed C23, C3, C6, C7, C8: 1uF, Capacitor_SMD:C_0805_2012Metric
- removed D1: ESD752, Package_TO_SOT_SMD:SOT-23
- removed D10, D2, D3, D4, D5, D6, D7, D8: LED, LED_SMD:LED_0805_2012Metric
- removed D9: SD12_SOD323, Diode_SMD:D_SOD-323
- removed H1, H2, H3, H4: M3, MountingHole:MountingHole_3.2mm_M3
- removed IC1: TPS56A37RPAR, UTSVT_Power:TPS56A37RPAR
- removed IC2: NPS4053GVH, UTSVT_Power:SOT95P275X110-6N
- removed J1: USB_C_Receptacle_PowerOnly_6P, UTSVT_Connectors:TYPEC31M17
- removed J10: GND_BANANA_OUT, UTSVT_Connectors:Banana_Jack_Horizontal
- removed J2: CC, Connector_PinHeader_2.54mm:PinHeader_1x03_P2.54mm_Vertical
- removed J3: 12V_OUT, UTSVT_Connectors:Molex_MicroFit3.0_1x2xP3.00mm_PolarizingPeg_Vertical
- removed J4: 5V_ISOOUT, UTSVT_Connectors:Molex_MicroFit3.0_1x2xP3.00mm_PolarizingPeg_Vertical
- removed J5: 5V_UNISOOUT, UTSVT_Connectors:Molex_MicroFit3.0_1x2xP3.00mm_PolarizingPeg_Vertical
- removed J6: 12V_OUT_PIN, Connector_PinHeader_2.54mm:PinHeader_1x02_P2.54mm_Vertical
- removed J7: 5V_ISOOUT_PIN, Connector_PinHeader_2.54mm:PinHeader_1x02_P2.54mm_Vertical
- removed J8: 5V_UNISOOUT_PIN, Connector_PinHeader_2.54mm:PinHeader_1x02_P2.54mm_Vertical
- removed J9: 12V_BANANA_OUT, UTSVT_Connectors:Banana_Jack_Horizontal
- removed L1: 5.6uH, UTSVT_Passive:INDPM110100X400N
- removed L2: 3.3uH, UTSVT_Passive:INDPM110100X400N
- removed NT1: NetTie_2, NetTie:NetTie-2_SMD_Pad2.0mm
- removed Q1: IRF9358TRPBF, UTSVT_ICs:SO8_IRF9358TRPBF_INF
- removed Q2: BSL308PEH6327XTSA1, Package_TO_SOT_SMD:SOT-23-6
- removed Q3: NVTR4503NT1G, Package_TO_SOT_SMD:SOT-23-3
- removed Q4, Q5: SI7149ADP-T1-GE3, UTSVT_ICs:POWERPAKSO-8
- removed R1, R17, R19, R2, R31, R33, R34: 10k, Resistor_SMD:R_0805_2012Metric
- removed R10, R35: 100k, Resistor_SMD:R_0805_2012Metric
- removed R11, R14, R16: 0, Resistor_SMD:R_0805_2012Metric
- removed R12, R13, R15: DNP, Resistor_SMD:R_0805_2012Metric
- removed R18, R20: 1k, Resistor_SMD:R_0805_2012Metric
- removed R21, R24, R29, R3, R32, R4, R5, R6, R7: 5.1k, Resistor_SMD:R_0805_2012Metric
- removed R22: 52.3k, Resistor_SMD:R_0805_2012Metric
- removed R23: 56k, Resistor_SMD:R_0805_2012Metric
- removed R25: 383k, Resistor_SMD:R_0805_2012Metric
- removed R26: 20k, Resistor_SMD:R_0805_2012Metric
- removed R27: 12k, Resistor_SMD:R_0805_2012Metric
- removed R28: 113k, Resistor_SMD:R_0805_2012Metric
- removed R30: 73.2k, Resistor_SMD:R_0805_2012Metric
- removed R36: 62k, Resistor_SMD:R_0805_2012Metric
- removed R8: 2.4k, Resistor_SMD:R_0805_2012Metric
- removed R9: 4.7k, Resistor_SMD:R_0805_2012Metric
- removed TP1: 12V_OUT_TP, TestPoint:TestPoint_Pad_D2.5mm
- removed TP10: VBUS_MIN_TP, TestPoint:TestPoint_Pad_D2.5mm
- removed TP11: VBUS_MAX_TP, TestPoint:TestPoint_Pad_D2.5mm
- removed TP12: ISNK_COARSE_TP, TestPoint:TestPoint_Pad_D2.5mm
- removed TP13: ISNK_FINE_TP, TestPoint:TestPoint_Pad_D2.5mm
- removed TP2: 5V_UNISO_TP, TestPoint:TestPoint_Pad_D2.5mm
- removed TP3: VBUS_USBIN, TestPoint:TestPoint_Pad_D2.5mm
- removed TP4: VBUS_TP, TestPoint:TestPoint_Pad_D2.5mm
- removed TP5: GND_TP, TestPoint:TestPoint_Pad_D2.5mm
- removed TP6: 5V_ISOOUT_TP, TestPoint:TestPoint_Pad_D2.5mm
- removed TP7: SAFE_5V_TP, TestPoint:TestPoint_Pad_D2.5mm
- removed TP8: GNDPWR_TP, TestPoint:TestPoint_Pad_D2.5mm
- removed TP9: 5V_BUCK_TP, TestPoint:TestPoint_Pad_D2.5mm
- removed U1: TVS2200DRV, Package_SON:WSON-6-1EP_2x2mm_P0.65mm_EP1x1.6mm
- removed U2: CYPD3177-24LQXQT, UTSVT_ICs:CYPD3177-24LQXQT_CYP
- removed U3: MAX16914AUB+, UTSVT_ICs:21-0061L_MXM
- removed U4: TPS562231DRLR, Package_TO_SOT_SMD:SOT-563
- removed U5: TPS2116DRL, Package_TO_SOT_SMD:SOT-583-8
- removed U6: TBA2-2411, Converter_DCDC:Converter_DCDC_TRACO_TBA2-xxxx_Single_THT
Routing:
- removed copper zone on F.Cu, net /VBUS_USBIN

Commit message: removed 12v output protection since buck already has OV
Parts:
- added C1: 3.3uF, Capacitor_SMD:C_0805_2012Metric, F.Cu at (217.5, 76.5)
- added C10: 0.1uF, Capacitor_SMD:C_0805_2012Metric, F.Cu at (143.1, 114.8)
- added C11: 10uF, Capacitor_SMD:C_2220_5750Metric, F.Cu at (132.3, 123.7)
- added C12: 0.1uF, Capacitor_SMD:C_0805_2012Metric, F.Cu at (143.1, 117.8)
- added C13: 22uF, Capacitor_SMD:C_1210_3225Metric, F.Cu at (148.2, 115.4)
- added C14: DNP, Capacitor_SMD:C_0805_2012Metric, F.Cu at (143.1, 120.8)
- added C15: 0.1uF, Capacitor_SMD:C_0805_2012Metric, F.Cu at (143.1, 123.8)
- added C16: 33pF, Capacitor_SMD:C_0805_2012Metric, F.Cu at (143.1, 126.8)
- added C17: 22uF, Capacitor_SMD:C_1210_3225Metric, F.Cu at (148.2, 119.6)
- added C18: 22uF, Capacitor_SMD:C_1210_3225Metric, F.Cu at (148.2, 123.9)
- added C19: 10uF, Capacitor_SMD:C_2220_5750Metric, F.Cu at (157.2, 116.7)
- added C2: 3.3uF, Capacitor_SMD:C_0805_2012Metric, F.Cu at (207.9, 76.5)
- added C20: 0.1uF, Capacitor_SMD:C_0805_2012Metric, F.Cu at (168.1, 114.8)
- added C21: 22uF, Capacitor_SMD:C_1210_3225Metric, F.Cu at (169.9, 103.5)
- added C22: 22uF, Capacitor_SMD:C_1210_3225Metric, F.Cu at (169.9, 107.8)
- added C3: 1uF, Capacitor_SMD:C_0805_2012Metric, F.Cu at (121.4, 109.5)
- added C4: 0.1uF, Capacitor_SMD:C_0805_2012Metric, F.Cu at (121.4, 112.5)
- added C5: 0.1uF, Capacitor_SMD:C_0805_2012Metric, F.Cu at (121.4, 115.5)
- added C6: 1uF, Capacitor_SMD:C_0805_2012Metric, F.Cu at (121.4, 118.5)
- added C7: 1uF, Capacitor_SMD:C_0805_2012Metric, F.Cu at (121.4, 121.6)
- added C8: 1uF, Capacitor_SMD:C_0805_2012Metric, F.Cu at (121.4, 124.6)
- added C9: 10uF, Capacitor_SMD:C_2220_5750Metric, F.Cu at (132.3, 116.7)
- added D1: ESD752, Package_TO_SOT_SMD:SOT-23, F.Cu at (152.7, 93.6)
- added D2: LED, LED_SMD:LED_0805_2012Metric, F.Cu at (111.6, 81.5)
- added D3: LED, LED_SMD:LED_0805_2012Metric, F.Cu at (111.6, 84.5)
- added D4: LED, LED_SMD:LED_0805_2012Metric, F.Cu at (111.6, 87.6)
- added D5: LED, LED_SMD:LED_0805_2012Metric, F.Cu at (111.6, 90.6)
- added D6: LED, LED_SMD:LED_0805_2012Metric, F.Cu at (111.6, 93.6)
- added D7: LED, LED_SMD:LED_0805_2012Metric, F.Cu at (111.6, 96.7)
- added D8: LED, LED_SMD:LED_0805_2012Metric, F.Cu at (112.2, 117.7)
- added D9: LED, LED_SMD:LED_0805_2012Metric, F.Cu at (130.3, 128.7)
- added F1: PTS120630V016, Fuse:Fuse_1206_3216Metric, F.Cu at (172.9, 60.0)
- added H1: M3, MountingHole:MountingHole_3.2mm_M3, F.Cu at (105.4, 53.5)
- added H2: M3, MountingHole:MountingHole_3.2mm_M3, F.Cu at (105.4, 61.5)
- added H3: M3, MountingHole:MountingHole_3.2mm_M3, F.Cu at (105.4, 69.4)
- added H4: M3, MountingHole:MountingHole_3.2mm_M3, F.Cu at (105.4, 77.4)
- added IC2: TPS56A37RPAR, UTSVT_Power:TPS56A37RPAR, F.Cu at (145.1, 104.3)
- added J1: USB_C_Receptacle_PowerOnly_6P, UTSVT_Connectors:TYPEC31M17, F.Cu at (212.8, 68.9)
- added J10: GND_BANANA_OUT, UTSVT_Connectors:Banana_Jack_Horizontal, F.Cu at (112.6, 67.3)
- added J2: CC, Connector_PinHeader_2.54mm:PinHeader_1x03_P2.54mm_Vertical, F.Cu at (148.1, 82.3)
- added J3: 12V_OUT, UTSVT_Connectors:Molex_MicroFit3.0_1x2xP3.00mm_PolarizingPeg_Vertical, F.Cu at (150.6, 53.1)
- added J4: 5V_ISOOUT, UTSVT_Connectors:Molex_MicroFit3.0_1x2xP3.00mm_PolarizingPeg_Vertical, F.Cu at (150.6, 60.4)
- added J5: 5V_UNISOOUT, UTSVT_Connectors:Molex_MicroFit3.0_1x2xP3.00mm_PolarizingPeg_Vertical, F.Cu at (150.6, 67.6)
- added J6: 12V_OUT_PIN, Connector_PinHeader_2.54mm:PinHeader_1x02_P2.54mm_Vertical, F.Cu at (134.2, 93.5)
- added J7: 5V_ISOOUT_PIN, Connector_PinHeader_2.54mm:PinHeader_1x02_P2.54mm_Vertical, F.Cu at (138.9, 93.5)
- added J8: 5V_UNISOOUT_PIN, Connector_PinHeader_2.54mm:PinHeader_1x02_P2.54mm_Vertical, F.Cu at (143.5, 93.5)
- added J9: 12V_BANANA_OUT, UTSVT_Connectors:Banana_Jack_Horizontal, F.Cu at (112.6, 52.1)
- added L1: 5.6uH, UTSVT_Passive:INDPM110100X400N, F.Cu at (135.1, 107.3)
- added L2: 4.7uH, UTSVT_Passive:INDPM110100X400N, F.Cu at (160.1, 107.3)
- added NT1: NetTie_2, NetTie:NetTie-2_SMD_Pad2.0mm, F.Cu at (145.7, 108.8)
- added Q1: IRF9358TRPBF, UTSVT_ICs:SO8_IRF9358TRPBF_INF, F.Cu at (105.7, 119.5)
- added Q2: BSL308PEH6327XTSA1, Package_TO_SOT_SMD:SOT-23-6, F.Cu at (123.5, 103.8)
- added R1: 10k, Resistor_SMD:R_0805_2012Metric, F.Cu at (116.0, 81.4)
- added R10: 0, Resistor_SMD:R_0805_2012Metric, F.Cu at (103.6, 111.7)
- added R11: DNP, Resistor_SMD:R_0805_2012Metric, F.Cu at (103.6, 114.7)
- added R12: DNP, Resistor_SMD:R_0805_2012Metric, F.Cu at (108.0, 102.9)
- added R13: 0, Resistor_SMD:R_0805_2012Metric, F.Cu at (108.0, 105.8)
- added R14: DNP, Resistor_SMD:R_0805_2012Metric, F.Cu at (108.0, 108.8)
- added R15: 0, Resistor_SMD:R_0805_2012Metric, F.Cu at (108.0, 111.7)
- added R16: 10k, Resistor_SMD:R_0805_2012Metric, F.Cu at (108.0, 114.7)
- added R17: 1k, Resistor_SMD:R_0805_2012Metric, F.Cu at (112.5, 102.9)
- added R18: 10k, Resistor_SMD:R_0805_2012Metric, F.Cu at (112.5, 105.8)
- added R19: 1k, Resistor_SMD:R_0805_2012Metric, F.Cu at (112.5, 108.8)
- added R2: 10k, Resistor_SMD:R_0805_2012Metric, F.Cu at (116.0, 84.4)
- added R20: 5.1k, Resistor_SMD:R_0805_2012Metric, F.Cu at (112.5, 111.7)
- added R21: 52.3k, Resistor_SMD:R_0805_2012Metric, F.Cu at (138.7, 114.7)
- added R22: 56k, Resistor_SMD:R_0805_2012Metric, F.Cu at (138.7, 117.7)
- added R23: 5.1k, Resistor_SMD:R_0805_2012Metric, F.Cu at (138.7, 120.6)
- added R24: 383k, Resistor_SMD:R_0805_2012Metric, F.Cu at (138.7, 123.6)
- added R25: 20k, Resistor_SMD:R_0805_2012Metric, F.Cu at (138.7, 126.5)
- added R26: 5.1k, Resistor_SMD:R_0805_2012Metric, F.Cu at (138.7, 129.5)
- added R27: 73.2k, Resistor_SMD:R_0805_2012Metric, F.Cu at (163.7, 114.7)
- added R28: 10k, Resistor_SMD:R_0805_2012Metric, F.Cu at (163.7, 117.7)
- added R29: 5.1k, Resistor_SMD:R_0805_2012Metric, F.Cu at (172.3, 51.0)
- added R3: 5.1k, Resistor_SMD:R_0805_2012Metric, F.Cu at (116.0, 87.3)
- added R30: 10k, Resistor_SMD:R_0805_2012Metric, F.Cu at (172.3, 54.0)
- added R31: 10k, Resistor_SMD:R_0805_2012Metric, F.Cu at (172.3, 56.9)
- added R4: 5.1k, Resistor_SMD:R_0805_2012Metric, F.Cu at (116.0, 90.3)
- added R5: 5.1k, Resistor_SMD:R_0805_2012Metric, F.Cu at (116.0, 93.2)
- added R6: 5.1k, Resistor_SMD:R_0805_2012Metric, F.Cu at (116.0, 96.2)
- added R7: 5.1k, Resistor_SMD:R_0805_2012Metric, F.Cu at (103.6, 102.9)
- added R8: 2.4k, Resistor_SMD:R_0805_2012Metric, F.Cu at (103.6, 105.8)
- added R9: 51k, Resistor_SMD:R_0805_2012Metric, F.Cu at (103.6, 108.8)
- added TP1: 12V_OUT_TP, TestPoint:TestPoint_Pad_D2.5mm, F.Cu at (120.5, 82.2)
- added TP10: VBUS_MIN_TP, TestPoint:TestPoint_Pad_D2.5mm, F.Cu at (116.9, 110.3)
- added TP11: VBUS_MAX_TP, TestPoint:TestPoint_Pad_D2.5mm, F.Cu at (116.9, 114.8)
- added TP12: ISNK_COARSE_TP, TestPoint:TestPoint_Pad_D2.5mm, F.Cu at (116.9, 119.4)
- added TP13: ISNK_FINE_TP, TestPoint:TestPoint_Pad_D2.5mm, F.Cu at (116.9, 123.9)
- added TP2: 5V_UNISO_TP, TestPoint:TestPoint_Pad_D2.5mm, F.Cu at (120.5, 86.8)
- added TP3: VBUS_USBIN, TestPoint:TestPoint_Pad_D2.5mm, F.Cu at (120.5, 91.3)
- added TP4: VBUS_TP, TestPoint:TestPoint_Pad_D2.5mm, F.Cu at (125.1, 82.2)
- added TP5: GND_TP, TestPoint:TestPoint_Pad_D2.5mm, F.Cu at (125.1, 86.8)
- added TP6: 5V_ISOOUT_TP, TestPoint:TestPoint_Pad_D2.5mm, F.Cu at (125.1, 91.3)
- added TP7: SAFE_5V_TP, TestPoint:TestPoint_Pad_D2.5mm, F.Cu at (129.6, 82.2)
- added TP8: GNDPWR_TP, TestPoint:TestPoint_Pad_D2.5mm, F.Cu at (129.6, 86.8)
- added TP9: 5V_BUCK_TP, TestPoint:TestPoint_Pad_D2.5mm, F.Cu at (129.6, 91.3)
- added U1: TVS2200DRV, Package_SON:WSON-6-1EP_2x2mm_P0.65mm_EP1x1.6mm, F.Cu at (152.4, 97.6)
- added U2: CYPD3177-24LQXQT, UTSVT_ICs:CYPD3177-24LQXQT_CYP, F.Cu at (117.8, 104.7)
- added U3: TPS562231DRLR, Package_TO_SOT_SMD:SOT-563, F.Cu at (167.8, 118.0)
- added U4: TPS2116DRL, Package_TO_SOT_SMD:SOT-583-8, F.Cu at (171.9, 63.7)
- added U5: TBA2-2411, Converter_DCDC:Converter_DCDC_TRACO_TBA2-xxxx_Single_THT, F.Cu at (167.9, 53.0)
Routing:
- added copper zone on F.Cu, net /VBUS
