File: 5v_buck_converter.kicad_sch (KiCad schematic)
At the start: 8 parts, among them U3 TPS562231DRLR

Commit message: started routing
Parts:
- C19: footprint Capacitor_SMD:C_2220_5750Metric -> Capacitor_SMD:C_0805_2012Metric; Manufacturer_Name KEMET -> Murata; Mouser Part Number C2220C106M5RACTU -> GRM21BR61H106KE43L
- C21: footprint Capacitor_SMD:C_1210_3225Metric -> Capacitor_SMD:C_0805_2012Metric; Manufacturer_Name Taiyo Yuden -> TDK; Mouser Part Number GMK325BJ226MM-P -> C2012X5R1V226M125AC
- C22: footprint Capacitor_SMD:C_1210_3225Metric -> Capacitor_SMD:C_0805_2012Metric; Manufacturer_Name Taiyo Yuden -> TDK; Mouser Part Number GMK325BJ226MM-P -> C2012X5R1V226M125AC; Vdc 50V -> 35V
Changed lines of the file:
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@@
 			)
 		)
-		(property "Footprint" "Capacitor_SMD:C_2220_5750Metric"
+		(property "Footprint" "Capacitor_SMD:C_0805_2012Metric"
 			(at 123.19 97.79 0)
 			(effects
@@
 			)
 		)
-		(property "Mouser Part Number" "C2220C106M5RACTU"
-			(at 123.19 97.79 0)
-			(effects
-				(font
-					(size 1.27 1.27)
-				)
-				(hide yes)
-			)
-		)
-		(property "Manufacturer_Name" "KEMET"
+		(property "Mouser Part Number" " GRM21BR61H106KE43L "
+			(at 123.19 97.79 0)
+			(effects
+				(font
+					(size 1.27 1.27)
+				)
+				(hide yes)
+			)
+		)
+		(property "Manufacturer_Name" "Murata"
 			(at 123.19 97.79 0)
 			(effects
@@
 			)
 		)
-		(property "Footprint" "Capacitor_SMD:C_1210_3225Metric"
+		(property "Footprint" "Capacitor_SMD:C_0805_2012Metric"
 			(at 180.6448 107.95 0)
 			(effects
@@
 			)
 		)
-		(property "Manufacturer_Name" "Taiyo Yuden"
-			(at 181.61 104.14 0)
-			(effects
-				(font
-					(size 1.27 1.27)
-				)
-				(hide yes)
-			)
-		)
-		(property "Mouser Part Number" " GMK325BJ226MM-P "
+		(property "Manufacturer_Name" "TDK"
+			(at 181.61 104.14 0)
+			(effects
+				(font
+					(size 1.27 1.27)
+				)
+				(hide yes)
+			)
+		)
+		(property "Mouser Part Number" "C2012X5R1V226M125AC"
 			(at 181.61 104.14 0)
 			(effects
@@
 			)
 		)
-		(property "Footprint" "Capacitor_SMD:C_1210_3225Metric"
+		(property "Footprint" "Capacitor_SMD:C_0805_2012Metric"
 			(at 190.8048 107.95 0)
 			(effects
@@
 			)
 		)
-		(property "Vdc" "50V"
+		(property "Vdc" "35V"
 			(at 191.77 104.14 0)
 			(effects
@@
 			)
 		)
-		(property "Manufacturer_Name" "Taiyo Yuden"
+		(property "Manufacturer_Name" "TDK"
 			(at 191.77 104.14 0)
 			(effects
@@
 			)
 		)
-		(property "Mouser Part Number" " GMK325BJ226MM-P "
+		(property "Mouser Part Number" "C2012X5R1V226M125AC"
 			(at 191.77 104.14 0)
 			(effects
