File: 5v_orring_isolator.kicad_sch (KiCad schematic)
At the start: 6 parts, among them U4 TPS2116DRL, U5 TBA2-2411

Commit message: i am jesus christ in the flesh.
Parts:
- F1: Mouser Part Number PTS120630V016 -> (none); P/N (none) -> PTS120630V016
- R29: Mouser Part Number CRCW08055K10FKEAC -> (none); P/N (none) -> CRCW08055K10FKEAC
- R30, R31: Mouser Part Number CRCW080510K0FKEAC -> (none); P/N (none) -> CRCW080510K0FKEAC
- U4: Mouser Part Number 595-TPS2116DRLR -> (none); P/N (none) -> TPS2116DRLR
- U5: Mouser Part Number 495-TBA2-2411 -> (none); P/N (none) -> TBA2-2411
Changed lines of the file:
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@@
 			)
 		)
-		(property "Mouser Part Number" "495-TBA2-2411"
+		(property "Mouser Part Number" ""
 			(at 191.77 101.6 0)
 			(effects
@@
 		)
 		(property "SnapEDA_Link" ""
+			(at 191.77 101.6 0)
+			(effects
+				(font
+					(size 1.27 1.27)
+				)
+				(hide yes)
+			)
+		)
+		(property "P/N" "TBA2-2411"
 			(at 191.77 101.6 0)
 			(effects
@@
 			)
 		)
-		(property "Mouser Part Number" "CRCW08055K10FKEAC "
+		(property "Mouser Part Number" ""
 			(at 83.82 96.52 0)
 			(effects
@@
 		)
 		(property "SnapEDA_Link" ""
+			(at 83.82 96.52 0)
+			(effects
+				(font
+					(size 1.27 1.27)
+				)
+				(hide yes)
+			)
+		)
+		(property "P/N" "CRCW08055K10FKEAC "
 			(at 83.82 96.52 0)
 			(effects
@@
 			)
 		)
-		(property "Mouser Part Number" "PTS120630V016"
+		(property "Mouser Part Number" ""
+			(at 208.28 99.06 0)
+			(effects
+				(font
+					(size 1.27 1.27)
+				)
+				(hide yes)
+			)
+		)
+		(property "P/N" "PTS120630V016"
 			(at 208.28 99.06 0)
 			(effects
@@
 			)
 		)
-		(property "Mouser Part Number" "595-TPS2116DRLR"
+		(property "Mouser Part Number" ""
 			(at 129.54 100.33 0)
 			(effects
@@
 		)
 		(property "SnapEDA_Link" ""
+			(at 129.54 100.33 0)
+			(effects
+				(font
+					(size 1.27 1.27)
+				)
+				(hide yes)
+			)
+		)
+		(property "P/N" "TPS2116DRLR"
 			(at 129.54 100.33 0)
 			(effects
@@
 			)
 		)
-		(property "Mouser Part Number" "CRCW080510K0FKEAC "
+		(property "Mouser Part Number" ""
 			(at 142.24 107.95 0)
 			(effects
@@
 		)
 		(property "SnapEDA_Link" ""
+			(at 142.24 107.95 0)
+			(effects
+				(font
+					(size 1.27 1.27)
+				)
+				(hide yes)
+			)
+		)
+		(property "P/N" "CRCW080510K0FKEAC"
 			(at 142.24 107.95 0)
 			(effects
@@
 			)
 		)
-		(property "Mouser Part Number" "CRCW080510K0FKEAC "
+		(property "Mouser Part Number" ""
 			(at 83.82 106.68 0)
 			(effects
@@
 			(at 83.82 106.68 0)
 			(effects
+				(font
+					(size 1.27 1.27)
+				)
+				(hide yes)
+			)
+		)
+		(property "P/N" "CRCW080510K0FKEAC"
+			(at 83.82 106.68 0)
+			(effects
