File: Boost Converter.kicad_sch (KiCad schematic)
At the start: 0 parts

Commit message: Finished initial SCH for boost converter
Parts:
- added C11: 4.7uF, symbol Device:C
- added C12, C7, C8: 0.1uF, symbol Device:C
- added C9: 2.2uF, symbol Device:C
- added IC1: LT8338JMSE#TRPBF, SOP50P490X110-11N, symbol LT8338JMSE:LT8338JMSE#TRPBF
- added L1: 20uH, symbol Device:L
- added R14: 1M, symbol Device:R_US
- added R15: 300k, symbol Device:R_US
- added R16: 93.1k, symbol Device:R_US
- added R17: 1.9M, symbol Device:R_US
- added R18: 2.0M, symbol Device:R_US
Connections:
- net VIN: now also C7.1, C8.1, IC1.1 (VIN), L1.2, R14.1
- new net: IC1.7 (RT), R16.2
- new net BST: C12.1, IC1.2 (BST)
- new net CTRL: IC1.9 (CTRL), R17.1, R18.2
- new net EN: IC1.8 (EN/UVLO), R14.2, R15.1
- new net GND: C11.2, C7.2, C8.2, C9.2, IC1.11 (GND), IC1.6 (SYNC/MODE), R15.2, R16.1, R18.1
- new net INTVCC: C9.1, IC1.10 (INTVCC), R17.2
- new net SW: C12.2, IC1.3 (SW_1), IC1.4 (SW_2), L1.1
- new net VOUT: C11.1, IC1.5 (VOUT)
Other:
- note added: "1V Falling edge for EN w/ 50 mV hysteresis 5V * (0.3/(1.0+0.3)) = 1.15 V ie. Cutoff when VIN < 5V"
- note added: "Burst Mode (Low IQ, low output ripple operation at light loads)"
- note added: "D(MAX) = (24-5)/24 = 0.79167 D(MIN) = (24-22)/24 = 0.08333"
- note added: "DECOUPLEING CAPS"
- note added: "ENABLE LOGIC"
- note added: "From Datasheet: deltaISW ~ 0.2 A L = (5 /(0.2 * 1MHz)) * 0.79167 L ~ 20 uH"
- note added: "INDUCTOR"
- note added: "INTVCC = 2.6V (2.0/(2.0+1.9))*2.6 = 1.3333V"
- note added: "Switching Freq fSW = 1MHz"
- note added: "VOUT = 18*VCTRL 24V = 18*1.3333V"
- note added: "VOUT CONTROL"
