File: STUSB4500.kicad_sch (KiCad schematic)
At the start: 27 parts, among them J2 TSW-104-07-T-S, Q1 STL6P3LLH6, Q2 STL6P3LLH6, U1 STUSB4500QTR

Commit message: Finished initial SCH for boost converter
Connections:
- net ALERT: no longer names the net of U1.19 (ALERT)
- no-connect marks 3 -> 4
Other:
- note added: "VBUS ~ 0 - 22 V"
- note added: "VDD ~ 4.1 - 22 V"
- note removed: "VBUS ~ 28 V"
- note removed: "VDD ~ 28 V"
Changed lines of the file:
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@@
 		)
 	)
-	(text "VBUS ~ 28 V"
+	(text "VBUS ~ 0 - 22 V"
 		(exclude_from_sim no)
-		(at 36.83 39.37 0)
+		(at 35.56 40.005 0)
 		(effects
 			(font
@@
 		)
 	)
-	(text "VDD ~ 28 V"
+	(text "VDD ~ 4.1 - 22 V"
 		(exclude_from_sim no)
 		(at 135.255 121.92 0)
@@
 	(no_connect
 		(at 122.555 161.29)
+	)
+	(no_connect
+		(at 88.265 161.29)
 	)
 	(wire
@@
 			"ADAAZgBDAHMANABZAEUAbQAzAE0AYQBTAHoAYwBDAGYAUwAxAFYAbABpAGcAMwB0ADQASwBRAEIA"
 			"bgBmAFQAcQBGAEYARwBqAFIARABDAE0AQgBVADMAVAB4AHgAZABlAGIAdAA2AEYAQwB3AGoASwBp"
-			"AHUANABlAC8AMw=="
+			"AHUANABlAC8AMwAAAAgAAAAAAAAA0M/cusoBAAABAAAAAAAAAAAAAAAAAAAApH87vAA8BICgLN66"
+			"ygEAAAMAAAAAAAAA4O7XusoBAAABAAAAAAAAAAAAAAAAAAAAq388vAA9BIBgJ966ygEAAAMAAAAA"
+			"AAAAAO/XusoBAAABAAAAAAAAAAAAAAAAAAAArn8xvAA+BIBAKd66ygEAAAMAAAAAAAAAIPLXusoB"
+			"AAABAAAAAAAAAAAAAAAAAAAArX8yvAA/BIDgKN66ygEAAAMAAAAAAAAAYPDXusoBAAABAAAAAAAA"
+			"AAAAAAAAAAAAsH83vABABIAAAAAAAAAAAAMAAAAAAAAAYGbeusoBAAABAAAAAAAAAAAAAAAAAAAA"
+			"t38ovABBBIAAM966ygEAAAMAAAAAAAAAIPXXusoBAAABAAAAAAAAAAAAAAAAAAAAun8tvABCBIAA"
+			"AAAAAAAAAAMAAAAAAAAA0DjeusoBAAABAAAAAAAAAAAAAAAAAAAAuX8uvABDBIBDOi9XSU5ET1dT"
+			"L2ZvbnRzXGNvdXJlZS5mb24AAAAAAAAAAAAAAAAAvH8jvABEBIAAAAAAAAAAAAgAAAAAAAAAUMrc"
+			"usoBAAABAAAAAAAAAAAAAAAAAAAAg38kvABFBIAAAAAAAAAAAAgAAAAAAAAAEMrcusoBAAABAAAA"
+			"AAAAAAAAAAAAAAAAhn8ZvABGBIAAAAAAAAAAAAMAAAAAAAAAgC7eusoBAAABAAAAAAAAAAAAAAAA"
+			"AAAAhX8avABHBIBDOi9XSU5ET1dTL2ZvbnRzXGNvdXJlZy5mb24AAAAAAAAAAAAAAAAAiH8fvABI"
+			"BIDQL966ygEAAAMAAAAAAAAA4PbXusoBAAABAAAAAAAAAAAAAAAAAAAAj38QvABJBIDQn9C+0LvR"
+			"g9C20LjRgNC90YvQuSDQmtGD0YDRgdC40LIAAAAAAAAAkn8VvABKBIAAAAAAAAAAAAMAAAAAAAAA"
+			"cGbeusoBAAABAAAAAAAAAAAAAAAAAAAAkX8WvABLBIAAAAAAAAAAAAMAAAAAAAAAcDjeusoBAAAB"
+			"AAAAAAAAAAAAAAAAAAAAlH8LvABMBIDAMN66ygEAAAMAAAAAAAAAgPjXusoBAAABAAAAAAAAAAAA"
+			"AAAAAAAAm38MvABNBIAAAAAAAAAAAAMAAAAAAAAAYGXeusoBAAABAAAAAAAAAAAAAAAAAAAAnn8B"
+			"vABOBIDgMd66ygEAAAMAAAAAAAAAwPvXusoBAAABAAAAAAAAAAAAAAAAAAAAnX8CvABPBIAAAAAA"
+			"AAAAAAMAAAAAAAAAUGXeusoBAAABAAAAAAAAAAAAAAAAAAAAYH4HvABQBIAAAAAAAAAAAAgAAAAA"
+			"AAAAUMbcusoBAAAAAAAAAAAAAAAAAAAAAAAAAAAAAAAAAAAAAAAAAAAAAAAAAAAAAAAAAAAAAAAA"
+			"AAAAAAAAAAAAAAAAAAAAAAAAAAAAAAAAAAAAAAAAAAAAAAAAAAAAAAAAAAAAAAAAAAAAAAAAAAAA"
+			"AAAAAAAAAAAAAAAAAAAAAAAAAAAAAAAAAAAAAAAAAAAAAAAAAAAAAAAAAAAAAAAAAAAAAAAAAAAA"
+			"AAAAAAAAAAAAAAAAAAAAAAAAAAAAAAAAAAAAAAAAAAAAAAAAAAAAAAAAAAAAAAAAAAAAAAAAAAAA"
+			"AAAAAAAAAAAAAAAAAAAAAAAAAAAAAAAAAAAAAAAAAAAAAAAAAAAAAAAAAAAAAAAAAAAAAAAAAAAA"
+			"AAAAAAAAAAAAAAAAAAAAAAAAAAAAAAAAAAAAAAAAAAAAAAAAAAAAAAAAAAAAAAAAAAAAAAAAAAAA"
+			"AAAAAAAAAAAAAAAAAAAAAAAAAAAAAAAAAAAAAAAAAAAAAAAAAAAAAAAAAAAAAAAAAAAAAAAAAAAA"
+			"AAAAAAAAAAAAAAAAAAAAAAAAAAAAAAAAAAAAAAAAAAAAAAAAAAAAAAAAAAAAAAAAAAAAAAAAAAAA"
+			"AAAAAAAAAAAAAAAAAAAAAAAAAAAAAAAAAAAAAAAAAAAAAAAAAAAAAAAAAAAAAAAAAAAAAAAAAAAA"
+			"AAAAAAAAAAAAAAAAAAAAAAAAAAAAAAAAAAAAAAAAAAAAAAAAAAAAAAAAAAAAAAAAAAAAAAAAAAAA"
+			"AAAAAAAAAAAAAAAAAAAAAAAAAAAAAAAAAAAAAAAAAAAAAAAAAAAAAAAAAAAAAAAAAAAAAAAAAAAA"
+			"AAAAAAAAAAAAAAAAAAAAAAAAAAAAAAAAAAAAAAAAAAAAAAAAAAAAAAAAAAAAAAAAAAAAAAAAAAAA"
+			"AAAAAAAAAAAAAAAAAAAAAAAAAAAAAAAAAAAAAAAAAAAAAAAAAAAAAAAAAAAAAAAAAAAAAAAAAAAA"
+			"AAAAAAAAAAAAAAAAAAAAAAAAAAAAAAAAAAAAAAAAAAAAAAAAAAAAAAAAAAAAAAAAAAAAAAAAAAAA"
+			"AAAAAAAAAAAAAAAAAAAAAAAAAAAAAAAAAAAAAAAAAAAAAAAAAAAAAAAAAAAAAAAAAAAAAAAAAAAA"
+			"AAAAAAAAAAAAAAAAAAAAAAAAAAAAAAAAAAAAAAAAAAAAAAAAAAAAAAAAAAAAAAAAAAAAAAAAAAAA"
+			"AAAAAAAAAAAAAAAAAAAAAAAAAAAAAAAAAAAAAAAAAAAAAAAAAAAAAAAAAAAAAAAAAAAAAAAAAAAA"
+			"AAAAAAAAAAAAAAAAAAAAAAAAAAAAAAAAAAAAAAAAAAAAAAAAAAAAAAAAAAAAAAAAAAAAAAAAAAAA"
+			"AAAAAAAAAAAAAA=="
 		)
 	)
@@
 		(effects
 			(font
-				(size 1.27 1.27)
-			)
-			(justify right bottom)
-		)
-	)
-	(label "ALERT"
-		(at 88.265 161.29 180)
-		(effects
-			(font
